File: KAKATA_RC433_V1/BOTONES_LATERALES.kicad_sch (KiCad schematic)
At the start: 12 parts, among them SW2 EVQPUC02K, SW3 EVQPUC02K, SW4 EVQPUC02K, SW5 EVQPUC02K

Commit message: Teminado ruteo Terminado colocacion de REF Verifacadas las conexiones Verificados todos los errores conocidos Verificados los de clerance
Parts:
- C18, C19, C20, C21: value C_0603 -> 100nF
- R15, R16, R17, R18: value R_0603 -> 22K; TOL (none) -> 1%
Connections:
- no-connect marks 0 -> 8

Commit message: Completado el BOM
Parts:
- C18, C19, C20, C21: LCSC Part (none) -> C14663
- R15, R16, R17, R18: LCSC Part (none) -> C114065
