File: KAKATA_RC433_V1/KAKATA_RC433_V1.kicad_sch (KiCad schematic)
At the start: 48 parts, among them U1 MKE04Z128VQH4, U10 74HC04, U2 MPU-6050_C24112, U3 433 MHz RF RECEIVER, U4 433 MHz TRANSMITTER, X1 X32258MOB4SI

Commit message: Actualizacion de componentes
Parts:
- removed C1, C2: CL10C120JB8NNNC, EasyEDA:C0603, symbol EasyEDA:CL10C120JB8NNNC
- removed H1: PROGRAMER, EasyEDA:HDR-TH_6P-P2.54-V-M, symbol EasyEDA:PZ2.54-1X6P-H25
- removed H2: I2C_AUX, EasyEDA:HDR-TH_2P-P2.54-V-M, symbol EasyEDA:PZ2.54-WV2P-H25
- removed H3: PWR, EasyEDA:HDR-TH_2P-P2.54-V-M, symbol EasyEDA:PZ2.54-WV2P-H25
- removed LED1, LED2, LED3, LED4, LED5, LED6: YLED0603R, EasyEDA:LED0603-FD, symbol EasyEDA:YLED0603R
- removed ON/OFF1: MT-0-123-D001-D000-LF, EasyEDA:SW-TH_3P-L13.1-W8.0-P4.70_MT-0-102-F001-T000-RS, symbol EasyEDA:MT-0-123-D001-D000-LF
- removed R1, R12, R13, R14, R15, R2, R3, R5, R6, R7, R8, R9: R_0603, PCM_Resistor_SMD_AKL:R_0603_1608Metric, symbol PCM_Resistor_US_AKL:R_0603
- removed U10: 74HC04, EasyEDA:SOIC-14_L8.7-W3.9-P1.27-LS6.0-BL, symbol EasyEDA:74HC04
- added BT1: 2477, EasyEDA:BAT-TH_2477, symbol EasyEDA:2477
- added C1, C13, C14, C15, C16, C17, C2: C_0603, Capacitor_SMD_AKL:C_0603_1608Metric, symbol PCM_Capacitor_US_AKL:C_0603
- added CN1: MG-JTAG-SWD6, MG_footprints:IDC-TH_6P-P2.54-V-R2-C3-S2.54, symbol MG_CONNECTORS:MG-JTAG-SWD6
- added R1, R14, R2, R5, R6, R7: R_0603, Resistor_SMD_AKL:R_0603_1608Metric, symbol Resistor_US_AKL:R_0603
- added SW1: ST-0-102-C03-N003-RS, EasyEDA:SW-TH_ST-0-102-C03-N003-RS, symbol EasyEDA:ST-0-102-C03-N003-RS
- added U6: HS96L03W2C03, EasyEDA:OLED-TH_L27.8-W27.2-P2.54_C9900033791, symbol EasyEDA:HS96L03W2C03
- added U7: LDL1117S33R, EasyEDA:SOT-223-4_L6.5-W3.5-P2.30-LS7.0-BR, symbol EasyEDA:LDL1117S33R
- C10, C11, C12, C3, C4, C5, C6, C7, C8, C9: footprint PCM_Capacitor_SMD_AKL:C_0603_1608Metric -> Capacitor_SMD_AKL:C_0603_1608Metric
- R10, R4: footprint PCM_Resistor_SMD_AKL:R_0603_1608Metric -> Resistor_SMD_AKL:R_0603_1608Metric
Connections:
- net +3.3V: now also U1.41 (VDD), U1.7 (VDD), C13.1, C14.1, C15.1, C16.1, CN1.2 (VCC), CN1.6 (VDD), R14.2, R5.2, R6.2, R7.2, U6.2 (VCC), U7.2 (VOUT), U7.4 (VOUT); no longer U1.9 (VREFL)
- net BTN_0: now also R5.1
- net BTN_1: now also R6.1
- net BTN_2: now also R7.1
- net BTN_3: now also R14.1
- net EXTAL: now also C2.1, R1.1
- net GND: now also U1.40 (VSS), U1.9 (VREFL), BT1.2 (-), C1.2, C13.2, C14.2, C15.2, C16.2, C17.2, C2.2, CN1.4 (GND), U6.1 (GND), U7.1 (GND)
- net I2C1_SCL: now also U6.3 (SCL)
- net I2C1_SDA: now also U6.4 (SDA)
- net RESET_b: now also CN1.5 (/RESET)
- net RF_IN: now also U3.5 (DO)
- net SWD_CLK: now also CN1.3 (SWD_CLK)
- net SWD_DIO: now also CN1.1 (SWD_DIO)
- net XTAL: now also R2.1
- net at X1.3: now also C1.1, R1.2, R2.2
- net LD1 renamed LED1
- new net: C17.1, SW1.3, U7.3 (VIN)
- new net: BT1.1 (+), SW1.2
- no-connect marks 2 -> 0
Other:
- added sheet BOTONES_LATERALES (BOTONES_LATERALES.kicad_sch)
- added sheet leds (untitled.kicad_sch)
- note added: "LCD"
- note removed: "SWITCH"
- moved on the sheet: BTN1, BTN3, C8, C9, U1

Commit message: Teminado ruteo Terminado colocacion de REF Verifacadas las conexiones Verificados todos los errores conocidos Verificados los de clerance
Parts:
- removed C14, C15, C16, C17: C_0603, Capacitor_SMD_AKL:C_0603_1608Metric, symbol PCM_Capacitor_US_AKL:C_0603
- removed CN1: MG-JTAG-SWD6, MG_footprints:IDC-TH_6P-P2.54-V-R2-C3-S2.54, symbol MG_CONNECTORS:MG-JTAG-SWD6
- removed R1, R2: R_0603, Resistor_SMD_AKL:R_0603_1608Metric, symbol Resistor_US_AKL:R_0603
- removed U1: MKE04Z128VQH4, EasyEDA:QFP-64_L14.0-W14.0-P0.80-LS17.2-BL, symbol EasyEDA:MKE04Z128VQH4
- removed X1: X32258MOB4SI, EasyEDA:CRYSTAL-SMD_4P-L3.2-W2.5-BL, symbol EasyEDA:X32258MOB4SI
- added C14, C15, C22: 10uF, Capacitor_SMD_AKL:C_0805_2012Metric, symbol Capacitor_AKL:C_0805
- added C17, C27: 47uF, Capacitor_SMD_AKL:CP_Elec_6.3x5.2, symbol Capacitor_AKL:CP_SMD_D6.3mm_H5.2mm
- added C23: 10nF, Capacitor_SMD_AKL:C_0603_1608Metric, symbol PCM_Capacitor_US_AKL:C_0603
- added C24, C26, C28: 100nF, Capacitor_SMD_AKL:C_0603_1608Metric, symbol PCM_Capacitor_US_AKL:C_0603
- added C25: 1uF, Capacitor_SMD_AKL:C_0603_1608Metric, symbol PCM_Capacitor_US_AKL:C_0603
- added D1, D3, D4: ESD5B5.0S, Diode_SMD_AKL:D_SOD-523, symbol Diode_TVS_AKL:ESD5B5.0S
- added D2, D5: B0540LW, Diode_SMD_AKL:D_SOD-123, symbol Diode_Schottky_AKL:B0540LW
- added JP1, JP2: SolderJumper_2_Open, Jumper:SolderJumper-2_P1.3mm_Open_RoundedPad1.0x1.5mm, symbol Jumper:SolderJumper_2_Open
- added L1: HPC4018BM-3R3M, EasyEDA:IND-SMD_L4.0-W4.0_HPC4030NF, symbol EasyEDA:HPC4018BM-3R3M
- added R1: 4.7k, Resistor_SMD_AKL:R_0603_1608Metric, symbol PCM_Resistor_US_AKL:R_0603
- added R19, R20: 5.1K, Resistor_SMD_AKL:R_0603_1608Metric, symbol Resistor_US_AKL:R_0603
- added R2: 4.7K, Resistor_SMD_AKL:R_0603_1608Metric, symbol PCM_Resistor_US_AKL:R_0603
- added R21, R22: 33R, Resistor_SMD_AKL:R_0603_1608Metric, symbol Resistor_US_AKL:R_0603
- added R23: 10K, Resistor_SMD_AKL:R_0603_1608Metric, symbol PCM_Resistor_US_AKL:R_0603
- added R24, R26: 100K, Resistor_SMD_AKL:R_0603_1608Metric, symbol PCM_Resistor_US_AKL:R_0603
- added R25, R27: 22K, Resistor_SMD_AKL:R_0603_1608Metric, symbol PCM_Resistor_US_AKL:R_0603
- added U1: MT3406, EasyEDA:SOT-23-5_L2.9-W1.6-P0.95-LS2.8-BR, symbol EasyEDA:MT3406
- added U8: ESP32-S3-WROOM-1U-N16R2, EasyEDA:WIRELM-SMD_ESP32-S3-WROOM-1U, symbol EasyEDA:ESP32-S3-WROOM-1U-N16R2
- added USB1: TYPE-C 16PIN 2MD(073), EasyEDA:USB-C-SMD_TYPE-C-6PIN-2MD-073, symbol EasyEDA:TYPE-C16PIN2MD(073)
- C1: value C_0603 -> 100nF; Dielec (none) -> X7R; TOL (none) -> +-10%; VOL (none) -> 4V
- C10, C11, C12, C13, C2, C3, C4, C5, C6, C7, C8, C9: value C_0603 -> 100nF; Dielec (none) -> X7R; TOL (none) -> +-10%; VOL (none) -> 50V
- R14, R5, R6, R7: value R_0603 -> 22K; TOL (none) -> 1%
Connections:
- net EXTAL is gone; now on an unnamed net: C2.1
- net I2C1_SCL is gone; now on net I2C_SCL: U6.3 (SCL)
- net I2C1_SDA is gone; now on net I2C_SDA: U6.4 (SDA)
- net +3.3V: now also C1.1, C17.1, C23.1, C27.1, JP1.2 (B), JP2.2 (B), R1.1, R2.1, R23.1, U8.2 (3V3); no longer C13.1, U7.2 (VOUT), U7.4 (VOUT)
- net ADC_JOY0_MD: now also C10.1, U8.5 (IO5); no longer C12.1
- net ADC_JOY0_MT: now also C12.1, U8.4 (IO4); no longer C8.1
- net ADC_JOY1_MD: now also C7.1, U8.39 (IO1); no longer C10.1
- net ADC_JOY1_MT: now also C8.1, U8.38 (IO2); no longer C9.1
- net BTNL1: now also U8.35 (IO42)
- net BTNL2: now also U8.34 (IO41)
- net BTNL3: now also U8.33 (IO40)
- net BTNL4: now also U8.32 (IO39)
- net BTN_0: now also C3.1, U8.17 (IO9); no longer C4.1
- net BTN_1: now also C4.1, U8.19 (IO11); no longer C11.1
- net BTN_2: now also C5.1, U8.18 (IO10); no longer C3.1
- net BTN_3: now also C11.1, U8.20 (IO12); no longer C5.1
- net GND: now also U2.1 (CLKIN), U2.11 (FSYNC), U2.25 (EP), U2.9 (AD0), C14.2, C15.2, C17.2, C22.2, C23.2, C24.2, C25.2, C26.2, C27.2, C28.2, D1.1 (K), D3.1 (K), D4.1 (K), R19.2, R20.2, R25.2, R27.2, U1.2 (GND), U8.1 (GND), U8.40 (GND), U8.41 (GND), USB1.1 (GND), USB1.12 (GND), USB1.13 (SHELL), USB1.14 (SHELL)
- net JOY0_BTN: now also U8.15 (IO3)
- net JOY1_BTN: now also C9.1, U8.16 (IO46); no longer C7.1
- net LED1: now also U8.26 (IO45)
- net LED2: now also U8.25 (IO48)
- net LED3: now also U8.24 (IO47)
- net LED4: now also U8.23 (IO21)
- net LED5: now also U8.22 (IO14)
- net LED6: now also U8.21 (IO13)
- net at SW1.3: now also BT1.1 (+), R26.1; no longer U7.3 (VIN)
- net at SW1.2: now also D5.2 (A); no longer BT1.1 (+)
- net at U2.10 (REGOUT): now also C24.1
- net INT_MPU: now reaches U2.12 (INT)
- net INT_MPU: now also U8.9 (IO16)
- net ANT: no longer names the net of U3.1 (ANT)
- net ENABLE renamed RF_ENABLE
- net RF_ENABLE: now also U8.8 (IO15)
- net GYRO_SCL renamed I2C_SCL
- net I2C_SCL: now also R1.2, U8.7 (IO7)
- net GYRO_SDA renamed I2C_SDA
- net I2C_SDA: now also R2.2, U8.6 (IO6)
- net RF_IN renamed DATA_RF_RECEIVED
- net DATA_RF_RECEIVED: now also U8.11 (IO18)
- net RF_OUT renamed DATA_RF_SEND
- net DATA_RF_SEND: now also U8.10 (IO17)
- new net: C25.1, R23.2, U8.3 (EN)
- new net: R20.1, USB1.10 (CC2)
- new net: R19.1, USB1.4 (CC1)
- new net: C13.1, JP1.1 (A), U7.2 (VOUT), U7.4 (VOUT)
- new net: C14.1, JP2.1 (A), L1.2, R24.1
- new net: R24.2, R25.1, U1.5 (FB)
- new net: L1.1, U1.3 (SW)
- new net USB_DN: D3.2 (A), R21.2, U8.13 (IO19)
- new net USB_DP: D4.2 (A), R22.2, U8.14 (IO20)
- new net VBAT: C28.1, R26.2, R27.1, U8.12 (IO8)
- new net VBUS: C22.1, D1.2 (A), D2.2 (A), USB1.11 (VBUS), USB1.2 (VBUS)
- new net con_dn: R21.1, USB1.5 (DN2), USB1.7 (DN1)
- new net con_dp: R22.1, USB1.6 (DP1), USB1.8 (DP2)
- new net vin: C15.1, C26.1, D2.1 (K), D5.1 (K), U1.1 (EN), U1.4 (VIN), U7.3 (VIN)
- no-connect marks 0 -> 34
Other:
- note added: "Battery Holder"
- note removed: "AUX_I2C"
- note removed: "BOTONES"
- note removed: "GYRO-I2C"
- note removed: "JOY0"
- note removed: "JOY1"
- note removed: "JOY_BTN"
- note removed: "LEDS"
- note removed: "RF_RECEIVER"
- note removed: "RF_TRANSMITER"
- note removed: "RF_TRANSMITTER"
- note removed: "‖"
- note removed: "‖ ‖"
- note removed: "‖ ‖ ‖"
- note removed: "‖ ‖ ‖ ‖"
- title: (none) -> KAKATA-RC433
- moved on the sheet: BT1, BTN1, BTN2, BTN3, BTN4, JOY0, JOY1, R10, R4, R5, U2, U3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

Commit message: Completado el BOM
Parts:
- C1, C24: LCSC Part (none) -> C519438
- C10, C11, C12, C13, C2, C26, C28, C3, C4, C5, C6, C7, C8, C9: LCSC Part (none) -> C14663
- C14, C15, C22: LCSC Part (none) -> C596327
- C17, C27: LCSC Part (none) -> C72522
- C23: LCSC Part (none) -> C100042
- C25: LCSC Part (none) -> C559769
- D1, D3, D4: LCSC Part (none) -> C93623
- D2, D5: LCSC Part (none) -> C53477639
- R1: value 4.7k -> 4.7K; LCSC Part (none) -> C99782
- R10, R4: value R_0603 -> 22K; LCSC Part (none) -> C114065
- R14, R25, R27, R5, R6, R7: LCSC Part (none) -> C114065
- R19, R20: LCSC Part (none) -> C105580
- R2: LCSC Part (none) -> C99782
- R21, R22: LCSC Part (none) -> C108661
- R23: LCSC Part (none) -> C98220
- R24, R26: LCSC Part (none) -> C14675
- U3, U4: now not fitted
