File: KAKATA_RC433_V1/untitled.kicad_sch (KiCad schematic)
At the start: 13 parts, among them U5 74HC04

Commit message: Teminado ruteo Terminado colocacion de REF Verifacadas las conexiones Verificados todos los errores conocidos Verificados los de clerance
Parts:
- added C16: 100nF, Capacitor_SMD_AKL:C_0603_1608Metric, symbol PCM_Capacitor_US_AKL:C_0603
- R11, R12, R13, R3, R8, R9: value R_0603 -> 220
Connections:
- net +3.3V: now also C16.1
- net GND: now also C16.2

Commit message: Completado el BOM
Parts:
- C16: LCSC Part (none) -> C14663
- R11, R12, R13, R3, R8, R9: LCSC Part (none) -> C107696
- U5: LCSC Part (none) -> C5590
